File: kicad/LocalDeck.kicad_pcb (KiCad board)
At the start: 2 copper layers, 124.5 x 102.9 mm, 74 parts, among them IC1 ESP32-C3-MINI-1-N4, J1 Conn_01x02_Pin, P1 USB_C_Receptacle_USB2.0, P2 USB_C_Receptacle_USB2.0, SW1 Boot, U1 AMS1117-3.3

Commit message: feat: Added programming Header
Parts:
- J1: value Conn_01x02_Pin -> Conn_Prog; footprint Connector_PinHeader_2.54mm:PinHeader_1x02_P2.54mm_Vertical -> LocalDeck Custom:ProgrammingHeader
- moved J1 5.39 mm to (42.7, 118.4), turned to -90 degrees
- moved D1 2.62 mm to (41.9, 109.5), turned to -90 degrees
Connections:
- J1 pad 1: GND -> /esp_boot
- J1 pad 2: VBUS -> GND
Routing:
- net /USB_D-: track 98.6 -> 134.3 mm, vias 5 -> 8
- net /esp_boot: track 35.2 -> 70.8 mm, vias 2 -> 4
- net /USB_D+: track 92.7 -> 104.3 mm, vias 5 -> 6
- net VBUS: track 154.1 -> 159.2 mm
- net Net-(LED10-DIN): track 15.4 -> 16.8 mm
- net +5V: track 562.7 -> 563.8 mm
- net Net-(LED6-DOUT): track 127.9 -> 127.3 mm
- net GND: vias 304 -> 302
- removed copper zone on F.Cu, net +5V
Other:
- board text added: "5V"
- board text added: "9"
- board text added: "D+"
- board text added: "D-"
- board text added: "G"
- board text removed: "VBUS-5V GND"

Commit message: chore(kicad): Added measurements & part numbers
Parts:
- moved R1 0.13 mm to (84.8, 109.9)
Routing:
- net /USB_D-: track 134.3 -> 124.9 mm
- net /col2: track 97.5 -> 96.1 mm
- net /led: track 73.4 -> 74.6 mm
- net /row3: track 266.9 -> 266.0 mm
- net /row1: track 251.6 -> 250.7 mm
- net /col5: track 132.7 -> 131.8 mm
- net /row2: track 280.1 -> 279.2 mm
- net /row0: track 236.8 -> 235.9 mm
- net +3.3V: track 65.4 -> 66.1 mm
- net GND: vias 302 -> 1139
Other:
- board text added: "©Allport-IT Ltd LB-Deck"
- board text removed: "2024-01"
- board text removed: "LB-Deck - ©Allport-IT Ltd - 2024-01"
